Commit message: Fix issue IntelRealSense/realsense-ros#2712

File: urdf/_d435.urdf.xacro (robot description, xacro)
@@ -8,5 +8,5 @@
 <robot name="sensor_d435" xmlns:xacro="http://ros.org/wiki/xacro">
   <!-- Includes -->
-  <xacro:include filename="$(find realsense2_description)/urdf/_d435.gazebo.xacro" />
+  <xacro:include filename="$(find realsense_gazebo_plugin)/urdf/_d435.gazebo.xacro" />
   <xacro:include filename="$(find realsense2_description)/urdf/_materials.urdf.xacro" />
   <xacro:include filename="$(find realsense2_description)/urdf/_usb_plug.urdf.xacro" />
@@ -54,5 +54,5 @@
           <origin xyz="${d435_zero_depth_to_glass + d435_glass_to_front} ${-d435_cam_depth_py} 0" rpy="${M_PI/2} 0 ${M_PI/2}"/>
           <geometry>
-            <mesh filename="package://realsense2_description/meshes/d435.dae" />
+            <mesh filename="file://$(find realsense2_description)/meshes/d435.dae" />
           </geometry>
         </xacro:if>

File: urdf/_d435i.urdf.xacro (robot description, xacro)
@@ -7,6 +7,6 @@
 -->
 <robot name="sensor_d435i" xmlns:xacro="http://ros.org/wiki/xacro">
-  <xacro:include filename="$(find realsense2_description)/urdf/_d435.urdf.xacro"/>
-  <xacro:include filename="$(find realsense2_description)/urdf/_d435i_imu_modules.urdf.xacro"/>
+  <xacro:include filename="$(find realsense_gazebo_plugin)/urdf/_d435.urdf.xacro"/>
+  <xacro:include filename="$(find realsense_gazebo_plugin)/urdf/_d435i_imu_modules.urdf.xacro"/>
   <xacro:macro name="sensor_d435i" params="parent *origin name:=camera use_nominal_extrinsics:=false add_plug:=false topics_ns:=camera publish_pointcloud:=false" >
     <xacro:sensor_d435 parent="${parent}" name="${name}" use_nominal_extrinsics="${use_nominal_extrinsics}" add_plug="${add_plug}" topics_ns="${topics_ns}" publish_pointcloud="${publish_pointcloud}">

File: urdf/test_d435_camera.urdf.xacro (robot description, xacro)
@@ -7,5 +7,5 @@
   <xacro:arg name="topics_ns" default="camera" />
   <xacro:arg name="publish_pointcloud" default="false" />
-  <xacro:include filename="$(find realsense2_description)/urdf/_d435.urdf.xacro" />
+  <xacro:include filename="$(find realsense_gazebo_plugin)/urdf/_d435.urdf.xacro" />
   <link name="base_link" />
   <xacro:sensor_d435 parent="base_link" use_nominal_extrinsics="$(arg use_nominal_extrinsics)" add_plug="$(arg add_plug)" use_mesh="$(arg use_mesh)" name="$(arg name)" topics_ns="$(arg topics_ns)" publish_pointcloud="$(arg publish_pointcloud)">

File: urdf/test_d435_multiple_cameras.urdf.xacro (robot description, xacro)
@@ -2,5 +2,5 @@
 <robot name="realsense2_camera" xmlns:xacro="http://ros.org/wiki/xacro">
   <xacro:arg name="use_nominal_extrinsics" default="false"/>
-  <xacro:include filename="$(find realsense2_description)/urdf/_d435.urdf.xacro" />
+  <xacro:include filename="$(find realsense_gazebo_plugin)/urdf/_d435.urdf.xacro" />
   <link name="base_link" />
   <xacro:sensor_d435 parent="base_link" name="camera1" use_nominal_extrinsics="$(arg use_nominal_extrinsics)">

File: urdf/test_d435i_camera.urdf.xacro (robot description, xacro)
@@ -6,5 +6,5 @@
   <xacro:arg name="publish_pointcloud" default="false" />
   <xacro:arg name="add_plug" default="false" />
-  <xacro:include filename="$(find realsense2_description)/urdf/_d435i.urdf.xacro"/>
+  <xacro:include filename="$(find realsense_gazebo_plugin)/urdf/_d435i.urdf.xacro"/>
   <link name="base_link" />
   <xacro:sensor_d435i name="$(arg name)" topics_ns="$(arg topics_ns)" parent="base_link" use_nominal_extrinsics="$(arg use_nominal_extrinsics)" publish_pointcloud="$(arg publish_pointcloud)" add_plug="$(arg add_plug)">
